File: PapoutPSM-HW.kicad_sch (KiCad schematic)
At the start: 24 parts, among them J1 53015-0510, U1 STM32G031F8P6, U2 SP3232EEY-L

Commit message: clean up some
Connections:
- net P_EMPTY: now also U1.12 (PA5); no longer U1.15 (PB0/PB1/PB2/PA8)
- net P_ERROR: now also U1.11 (PA4); no longer U1.16 (PA11_[PA9])
- net P_INHIBIT: now also U1.16 (PA11_[PA9]); no longer U1.11 (PA4)
- net P_OUT_PULSE: now also U1.13 (PA6); no longer U1.14 (PA7)
- net P_PULSE: now also U1.14 (PA7); no longer U1.13 (PA6)
- net P_RESET: now also U1.15 (PB0/PB1/PB2/PA8); no longer U1.12 (PA5)
Changed lines of the file:
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@@
     (title "Main Block")
     (date "2021-07-30")
-    (rev "0.1")
+    (rev "0.4")
     (company "Korean Paper Dispenser Parallel to Serial Adapter Module")
     (comment 1 "Features : 24V -> 12V, RS232, STM32G030")
@@
     (effects (font (size 1.27 1.27)) (justify right bottom))
   )
-  (label "P_ERROR" (at 139.7 45.72 180)
+  (label "P_INHIBIT" (at 137.16 45.72 180)
     (effects (font (size 1.27 1.27)) (justify right bottom))
   )
-  (label "P_EMPTY" (at 139.7 48.26 180)
+  (label "P_RESET" (at 137.16 48.26 180)
     (effects (font (size 1.27 1.27)) (justify right bottom))
   )
-  (label "P_OUT_PULSE" (at 139.7 50.8 180)
+  (label "P_PULSE" (at 137.16 50.8 180)
     (effects (font (size 1.27 1.27)) (justify right bottom))
   )
-  (label "P_PULSE" (at 139.7 53.34 180)
+  (label "P_OUT_PULSE" (at 137.16 53.34 180)
     (effects (font (size 1.27 1.27)) (justify right bottom))
   )
-  (label "P_RESET" (at 139.7 55.88 180)
+  (label "P_EMPTY" (at 137.16 55.88 180)
     (effects (font (size 1.27 1.27)) (justify right bottom))
   )
-  (label "P_INHIBIT" (at 139.7 58.42 180)
+  (label "P_ERROR" (at 137.16 58.42 180)
     (effects (font (size 1.27 1.27)) (justify right bottom))
   )
@@
       (effects (font (size 1.27 1.27)) (justify left top))
     )
-    (pin "P_ERROR" output (at 142.24 45.72 180)
-      (effects (font (size 1.27 1.27)) (justify left))
-    )
-    (pin "P_PULSE" input (at 142.24 53.34 180)
-      (effects (font (size 1.27 1.27)) (justify left))
-    )
-    (pin "P_OUT_PULSE" output (at 142.24 50.8 180)
-      (effects (font (size 1.27 1.27)) (justify left))
-    )
-    (pin "P_EMPTY" output (at 142.24 48.26 180)
-      (effects (font (size 1.27 1.27)) (justify left))
-    )
-    (pin "P_RESET" input (at 142.24 55.88 180)
-      (effects (font (size 1.27 1.27)) (justify left))
-    )
-    (pin "P_INHIBIT" input (at 142.24 58.42 180)
-      (effects (font (size 1.27 1.27)) (justify left))
-    )
+    (pin "P_ERROR" output (at 142.24 58.42 180)
+      (effects (font (size 1.27 1.27)) (justify left))
+    )
+    (pin "P_PULSE" input (at 142.24 50.8 180)
+      (effects (font (size 1.27 1.27)) (justify left))
+    )
+    (pin "P_OUT_PULSE" output (at 142.24 53.34 180)
+      (effects (font (size 1.27 1.27)) (justify left))
+    )
+    (pin "P_EMPTY" output (at 142.24 55.88 180)
+      (effects (font (size 1.27 1.27)) (justify left))
+    )
+    (pin "P_RESET" input (at 142.24 48.26 180)
+      (effects (font (size 1.27 1.27)) (justify left))
+    )
+    (pin "P_INHIBIT" input (at 142.24 45.72 180)
+      (effects (font (size 1.27 1.27)) (justify left))
+    )

Commit message: some layout changed (sizeup for later 2layer conversion)
Parts:
- added C4: 100nF, Capacitor_SMD:C_0402_1005Metric, symbol Device:C
- added U2: MB85RS64, Package_SO:SOIC-8_3.9x4.9mm_P1.27mm, symbol Memory_NVRAM:MB85RS64
- renumbered C4 to C5, C5 to C6, C6 to C7, C7 to C8, C8 to C9, U2 to U3
Connections:
- net +3V3: now also C4.1, U2.8 (VDD)
- net GND: now also C4.2, U2.4 (GND); no longer U1.17 (PA12_[PA10]), U1.7 (PA0), U1.8 (PA1)
- net TEST_POINT: no longer U1.20 (PB3/PB4/PB5/PB6)
- new net FRAM_MISO: U1.20 (PB3/PB4/PB5/PB6), U2.2 (SO)
- new net FRAM_MOSI: U1.17 (PA12_[PA10]), U2.5 (SI)
- new net FRAM_SCK: U1.8 (PA1), U2.6 (SCK)
