File: PapoutPSM-HW.kicad_sch (KiCad schematic)
At the start: 17 parts, among them J1 Conn_01x05, J2 53014-1010, SW1 SW_DIP_x04

Commit message: v1
Parts:
- removed C3: 100nF, Capacitor_SMD:C_0402_1005Metric, symbol Device:C
- removed J2: 53014-1010, Connector_Extended_Molex_53014:Molex_MicroBlade_53014-1000_1x10_P2.00mm_Vertical, symbol Connector_Generic:Conn_01x10
- removed R3, R4, R5, R6: 10k, Resistor_SMD:R_0402_1005Metric, symbol Device:R_US
- removed R7, R8, R9: 100, Resistor_SMD:R_0402_1005Metric, symbol Device:R_US
- removed SW1: SW_DIP_x04, Button_Switch_THT:SW_DIP_SPSTx04_Slide_9.78x12.34mm_W7.62mm_P2.54mm, symbol Switch:SW_DIP_x04
- added C4, C5, C6, C7, C8: 100nF, Capacitor_SMD:C_0402_1005Metric, symbol Device:C
- added D1, D2: LED_RED, LED_SMD:LED_0805_2012Metric, symbol Device:LED
- added H1, H2, H3, H4: MountingHole, MountingHole:MountingHole_4.3mm_M4_ISO14580_Pad, symbol Mechanical:MountingHole
- added TP1: TestPoint, TestPoint:TestPoint_Pad_D1.0mm, symbol Connector:TestPoint
- added U1: STM32G030F6, Package_SO:TSSOP-20_4.4x6.5mm_P0.65mm, symbol STM32G0:STM32G030F6
- added U2: SP3232EEY-L, Package_SO:TSSOP-16_4.4x5mm_P0.65mm, symbol Interface_UART_Extended:SP3232EEY-L
- J1: footprint Connector_Extended_Molex_53014:Molex_MicroBlade_53014-0500_1x05_P2.00mm_Vertical -> Molex-53015:Molex_MicroBlade_53015-0500_1x05_P2.00mm_Right
- R1, R2: value 10k -> 4.7k; LCSC Part C25744 -> C25900; MFR.Part# 0402WGF1002TCE -> 0402WGF4701TCE; ODR.Part# RES 10k 1005 -> RES 4.7k 1005
- renumbered C4 to C3
Connections:
- net +3V3: now also DEBUG1.2 (Pin_2), C4.1, C7.2, U1.4 (VDD/VDDA), U2.16 (VCC); no longer R1.1, R2.1
- net GND: now also C4.2, C8.2, D1.1 (K), D2.1 (K), U1.17 (PA12_[PA10]), U1.3 (PC15-OSC32_OUT), U1.5 (VSS/VSSA), U1.7 (PA0), U1.8 (PA1), U2.10 (T2IN), U2.15 (GND), U2.8 (R2IN)
- net SWCLK: now reaches DEBUG1.5 (Pin_5)
- net SWCLK: now also U1.19 (PA15/PA14-BOOT0)
- net SWDIO: now reaches DEBUG1.3 (Pin_3)
- net SWDIO: now also U1.18 (PA13)
- net R_TXD: now reaches J1.4 (Pin_4)
- net R_TXD: now also U2.11 (T1IN)
- net R_RXD: now reaches J1.5 (Pin_5)
- net R_RXD: now also U2.12 (R1OUT)
- net EN renamed NRST
- net NRST: now also U1.6 (~RST); no longer R1.2
- net IO9: no longer names the net of R2.2
- net IO9: now also D2.2 (A); no longer DEBUG1.6 (Pin_6)
- new net: C5.1, U2.3 (C1-)
- new net: C5.2, U2.1 (C1+)
- new net: C8.1, U2.6 (V-)
- new net: C7.1, U2.2 (V+)
- new net: D1.2 (A), R1.2
- new net: C6.2, U2.4 (C2+)
- new net: C6.1, U2.5 (C2-)
- new net LED0: R1.1, U1.1 (PB7/PB8)
- new net LED1: R2.1, U1.2 (PB9/PC14-OSC32_IN)
- new net M_RX: U1.10 (PA3), U2.14 (T1OUT)
- new net M_TX: U1.9 (PA2), U2.13 (R1IN)
- new net P_EMPTY: U1.12 (PA5)
- new net P_ERROR: U1.11 (PA4)
- new net P_INHIBIT: U1.16 (PA11_[PA9])
- new net P_OUT_PULSE: U1.13 (PA6)
- new net P_PULSE: U1.14 (PA7)
- new net P_RESET: U1.15 (PB0/PB1/PB2/PA8)
- new net TEST_POINT: TP1.1, U1.20 (PB3/PB4/PB5/PB6)
- no-connect marks 0 -> 3
Other:
- sheet Parallel_IO ports: added P_EMPTY, P_ERROR, P_INHIBIT, P_OUT_PULSE, P_PULSE, P_RESET; removed none
- moved on the sheet: C2, C3, DEBUG1, J1

Commit message: stuff
Parts:
- C1: value 22uF -> 4.7uF; footprint Capacitor_SMD:C_0805_2012Metric -> Capacitor_SMD:C_0402_1005Metric; LCSC Part C45783 -> C1525; MFR.Part# CL21A226MAQNNNE -> CL05B104KO5NNNC; ODR.Part# CAP 22uF 25V 2012 -> CAP 100nF 1005; Packaging 2012 -> 1005
Changed lines of the file:
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@@
       (effects (font (size 1.27 1.27)) (justify left))
     )
-    (property "Value" "22uF" (id 1) (at 30.861 37.973 0)
-      (effects (font (size 1.27 1.27)) (justify left))
-    )
-    (property "Footprint" "Capacitor_SMD:C_0805_2012Metric" (id 2) (at 28.9052 40.64 0)
+    (property "Value" "4.7uF" (id 1) (at 30.861 37.973 0)
+      (effects (font (size 1.27 1.27)) (justify left))
+    )
+    (property "Footprint" "Capacitor_SMD:C_0402_1005Metric" (id 2) (at 28.9052 40.64 0)
       (effects (font (size 1.27 1.27)) hide)
     )
@@
       (effects (font (size 1.27 1.27)) hide)
     )
-    (property "LCSC Part" "C45783" (id 4) (at 27.94 36.83 0)
-      (effects (font (size 1.27 1.27)) hide)
-    )
-    (property "MFR.Part#" "CL21A226MAQNNNE" (id 5) (at 27.94 36.83 0)
+    (property "LCSC Part" "C1525" (id 4) (at 27.94 36.83 0)
+      (effects (font (size 1.27 1.27)) hide)
+    )
+    (property "MFR.Part#" "CL05B104KO5NNNC" (id 5) (at 27.94 36.83 0)
       (effects (font (size 1.27 1.27)) hide)
     )
@@
       (effects (font (size 1.27 1.27)) hide)
     )
-    (property "ODR.Part#" "CAP 22uF 25V 2012" (id 8) (at 30.48 40.64 0)
-      (effects (font (size 1.27 1.27)) (justify left) hide)
-    )
-    (property "Packaging" "2012" (id 9) (at 27.94 36.83 0)
+    (property "ODR.Part#" "CAP 100nF 1005" (id 8) (at 27.94 36.83 0)
+      (effects (font (size 1.27 1.27)) hide)
+    )
+    (property "Packaging" "1005" (id 9) (at 27.94 36.83 0)
       (effects (font (size 1.27 1.27)) hide)
     )
@@
       (reference "#SYM1") (unit 1) (value "SYM_Arrow45_Small") (footprint "Symbol_Extended:LamudaEE-12.8x7.9mm")
     )
-    (path "/270d8768-ac22-4e63-a610-77bb5a66f5be"
-      (reference "C1") (unit 1) (value "22uF") (footprint "Capacitor_SMD:C_0805_2012Metric")
+    (path "/d7f6a424-56ee-4c03-88f2-634b72b69d74"
+      (reference "C1") (unit 1) (value "4.7uF") (footprint "Capacitor_SMD:C_0402_1005Metric")
     )
     (path "/2df5bce9-42e4-410e-af77-e78cd3807d23"

Commit message: update bom
Parts:
- added SYM1: SYM_Arrow_Tiny, Symbol_Extended:LamudaEE-12.8x7.9mm, symbol Graphic:SYM_Arrow_Tiny
- D1, D2: value LED_RED -> LED GREEN; LCSC Part C84256 -> C2297; MFR.Part# FC-2012HRK-620D -> KT-0805G; ODR.Part# LED RED 2012 -> LED GREEN 2012
- H1, H2, H3, H4: Mount (none) -> N/C
- J1: value Conn_01x05 -> 53015-0510; MFR.Part# (none) -> 53015-0510; Manufacturer (none) -> Molex; Mount (none) -> TH; ODR.Part# (none) -> 53015-0510; Packaging (none) -> DIP-5-2mm; Supplier (none) -> Asian Supplier
Changed lines of the file:
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@@
     (effects (font (size 1.27 1.27)) (justify right bottom))
+  )
+  (symbol (lib_id "Graphic:SYM_Arrow_Tiny") (at 213.36 124.46 0) (unit 1)
+    (in_bom no) (on_board yes)
+    (property "Reference" "SYM1" (id 0) (at 213.36 122.936 0))
+    (property "Value" "SYM_Arrow_Tiny" (id 1) (at 213.614 125.73 0)
+      (effects (font (size 1.27 1.27)) hide)
+    )
+    (property "Footprint" "Symbol_Extended:LamudaEE-12.8x7.9mm" (id 2) (at 236.22 124.46 0))
+    (property "Datasheet" "~" (id 3) (at 213.36 124.46 0)
+      (effects (font (size 1.27 1.27)) hide)
+    )
   )
   (symbol (lib_id "power:+3V3") (at 39.37 33.02 0) (unit 1)
@@
     (pin "1")
   )
-  (symbol (lib_id "Graphic:SYM_Arrow45_Small") (at 213.36 124.46 0) (unit 1)
-    (in_bom yes) (on_board yes) (fields_autoplaced)
-    (property "Reference" "#SYM1" (id 0) (at 217.678 123.444 0)
-      (effects (font (size 1.27 1.27)) hide)
-    )
-    (property "Value" "SYM_Arrow45_Small" (id 1) (at 213.36 126.746 0)
-      (effects (font (size 1.27 1.27)) hide)
-    )
-    (property "Footprint" "Symbol_Extended:LamudaEE-12.8x7.9mm" (id 2) (at 213.36 124.46 0)
-      (effects (font (size 1.27 1.27)) hide)
-    )
-    (property "Datasheet" "~" (id 3) (at 213.36 124.46 0)
-      (effects (font (size 1.27 1.27)) hide)
-    )
-  )
   (symbol (lib_id "Mechanical:MountingHole") (at 213.36 130.81 0) (unit 1)
     (in_bom yes) (on_board yes) (fields_autoplaced)
@@
       (effects (font (size 1.27 1.27)) hide)
     )
+    (property "Mount" "N/C" (id 4) (at 213.36 130.81 0)
+      (effects (font (size 1.27 1.27)) hide)
+    )
   )
   (symbol (lib_id "Mechanical:MountingHole") (at 213.36 138.43 0) (unit 1)
@@
       (effects (font (size 1.27 1.27)) hide)
     )
+    (property "Mount" "N/C" (id 4) (at 213.36 138.43 0)
+      (effects (font (size 1.27 1.27)) hide)
+    )
   )
   (symbol (lib_id "Mechanical:MountingHole") (at 237.49 130.81 0) (unit 1)
@@
       (effects (font (size 1.27 1.27)) hide)
     )
+    (property "Mount" "N/C" (id 4) (at 237.49 130.81 0)
+      (effects (font (size 1.27 1.27)) hide)
+    )
   )
   (symbol (lib_id "Mechanical:MountingHole") (at 237.49 138.43 0) (unit 1)
@@
     )
     (property "Datasheet" "~" (id 3) (at 237.49 138.43 0)
+      (effects (font (size 1.27 1.27)) hide)
+    )
+    (property "Mount" "N/C" (id 4) (at 237.49 138.43 0)
       (effects (font (size 1.27 1.27)) hide)
     )
@@
     (in_bom yes) (on_board yes)
     (property "Reference" "D1" (id 0) (at 156.3878 69.723 0))
-    (property "Value" "LED_RED" (id 1) (at 156.3878 72.0344 0))
+    (property "Value" "LED GREEN" (id 1) (at 156.3878 72.0344 0))
     (property "Footprint" "LED_SMD:LED_0805_2012Metric" (id 2) (at 156.21 76.2 0)
       (effects (font (size 1.27 1.27)) hide)
     )
-    (property "Datasheet" "Foshan-NationStar-Optoelectronics-FC-2012HRK-620D_C84256.pdf" (id 3) (at 156.21 76.2 0)
-      (effects (font (size 1.27 1.27)) hide)
-    )
-    (property "LCSC Part" "C84256" (id 4) (at 156.21 76.2 0)
-      (effects (font (size 1.27 1.27)) hide)
-    )
-    (property "MFR.Part#" "FC-2012HRK-620D" (id 5) (at 156.21 76.2 0)
+    (property "Datasheet" "https://datasheet.lcsc.com/lcsc/1806151820_Hubei-KENTO-Elec-C2297_C2297.pdf" (id 3) (at 156.21 76.2 0)
+      (effects (font (size 1.27 1.27)) hide)
+    )
+    (property "LCSC Part" "C2297" (id 4) (at 156.21 76.2 0)
+      (effects (font (size 1.27 1.27)) hide)
+    )
+    (property "MFR.Part#" "KT-0805G" (id 5) (at 156.21 76.2 0)
       (effects (font (size 1.27 1.27)) hide)
     )
@@
       (effects (font (size 1.27 1.27)) hide)
     )
-    (property "ODR.Part#" "LED RED 2012" (id 8) (at 156.21 76.2 0)
+    (property "ODR.Part#" "LED GREEN 2012" (id 8) (at 156.21 76.2 0)
       (effects (font (size 1.27 1.27)) hide)
     )
@@
     (in_bom yes) (on_board yes)
     (property "Reference" "D2" (id 0) (at 156.3878 80.518 0))
-    (property "Value" "LED_RED" (id 1) (at 156.3878 82.8294 0))
+    (property "Value" "LED GREEN" (id 1) (at 156.3878 82.8294 0))
     (property "Footprint" "LED_SMD:LED_0805_2012Metric" (id 2) (at 156.21 86.995 0)
       (effects (font (size 1.27 1.27)) hide)
     )
-    (property "Datasheet" "Foshan-NationStar-Optoelectronics-FC-2012HRK-620D_C84256.pdf" (id 3) (at 156.21 86.995 0)
-      (effects (font (size 1.27 1.27)) hide)
-    )
-    (property "LCSC Part" "C84256" (id 4) (at 156.21 86.995 0)
-      (effects (font (size 1.27 1.27)) hide)
-    )
-    (property "MFR.Part#" "FC-2012HRK-620D" (id 5) (at 156.21 86.995 0)
+    (property "Datasheet" "https://datasheet.lcsc.com/lcsc/1806151820_Hubei-KENTO-Elec-C2297_C2297.pdf" (id 3) (at 156.21 86.995 0)
+      (effects (font (size 1.27 1.27)) hide)
+    )
+    (property "LCSC Part" "C2297" (id 4) (at 156.21 86.995 0)
+      (effects (font (size 1.27 1.27)) hide)
+    )
+    (property "MFR.Part#" "KT-0805G" (id 5) (at 156.21 86.995 0)
       (effects (font (size 1.27 1.27)) hide)
     )
@@
       (effects (font (size 1.27 1.27)) hide)
     )
-    (property "ODR.Part#" "LED RED 2012" (id 8) (at 156.21 86.995 0)
+    (property "ODR.Part#" "LED GREEN 2012" (id 8) (at 156.21 86.995 0)
       (effects (font (size 1.27 1.27)) hide)
     )
@@
     (in_bom yes) (on_board yes) (fields_autoplaced)
     (property "Reference" "J1" (id 0) (at 232.918 83.82 0))
-    (property "Value" "Conn_01x05" (id 1) (at 232.918 86.36 0))
+    (property "Value" "53015-0510" (id 1) (at 232.918 86.36 0))
     (property "Footprint" "Molex-53015:Molex_MicroBlade_53015-0500_1x05_P2.00mm_Right" (id 2) (at 234.95 95.25 0)
       (effects (font (size 1.27 1.27)) hide)
     )
-    (property "Datasheet" "~" (id 3) (at 234.95 95.25 0)
+    (property "Datasheet" "https://www.molex.com/pdm_docs/sd/530140410_sd.pdf" (id 3) (at 234.95 95.25 0)
+      (effects (font (size 1.27 1.27)) hide)
+    )
+    (property "MFR.Part#" "53015-0510" (id 4) (at 234.95 95.25 0)
+      (effects (font (size 1.27 1.27)) hide)
+    )
+    (property "Manufacturer" "Molex" (id 5) (at 234.95 95.25 0)
+      (effects (font (size 1.27 1.27)) hide)
+    )
+    (property "Mount" "TH" (id 6) (at 234.95 95.25 0)
+      (effects (font (size 1.27 1.27)) hide)
+    )
+    (property "ODR.Part#" "53015-0510" (id 7) (at 234.95 95.25 0)
+      (effects (font (size 1.27 1.27)) hide)
+    )
+    (property "Packaging" "DIP-5-2mm" (id 8) (at 234.95 95.25 0)
+      (effects (font (size 1.27 1.27)) hide)
+    )
+    (property "Supplier" "Asian Supplier" (id 9) (at 234.95 95.25 0)
       (effects (font (size 1.27 1.27)) hide)
     )
@@
       (reference "#PWR064") (unit 1) (value "GND") (footprint "")
     )
-    (path "/63424375-b7c3-41c1-95b7-8b13a0e766cd"
-      (reference "#SYM1") (unit 1) (value "SYM_Arrow45_Small") (footprint "Symbol_Extended:LamudaEE-12.8x7.9mm")
-    )
     (path "/d7f6a424-56ee-4c03-88f2-634b72b69d74"
       (reference "C1") (unit 1) (value "4.7uF") (footprint "Capacitor_SMD:C_0402_1005Metric")
@@
     )
     (path "/8a2bfc1f-24c7-490b-b3d7-517ff14522dd"
-      (reference "D1") (unit 1) (value "LED_RED") (footprint "LED_SMD:LED_0805_2012Metric")
+      (reference "D1") (unit 1) (value "LED GREEN") (footprint "LED_SMD:LED_0805_2012Metric")
     )
     (path "/08c0b325-5774-43ee-856e-b47604aa5ed2"
-      (reference "D2") (unit 1) (value "LED_RED") (footprint "LED_SMD:LED_0805_2012Metric")
+      (reference "D2") (unit 1) (value "LED GREEN") (footprint "LED_SMD:LED_0805_2012Metric")
     )
     (path "/6dfaa3f9-076c-470d-9afe-3e64c474240c/03862d63-1ff0-4c5f-bf48-1bab02691ca8"
-      (reference "D3") (unit 1) (value "LED_RED") (footprint "LED_SMD:LED_0805_2012Metric")
+      (reference "D3") (unit 1) (value "LED GREEN") (footprint "LED_SMD:LED_0805_2012Metric")
     )
     (path "/6dfaa3f9-076c-470d-9afe-3e64c474240c/9cb128cd-6ce1-4dfc-b3bf-bc9d2ec9877c"
@@
     )
     (path "/fb8c28c8-63b1-4364-a6f7-7612e8ee157e"
-      (reference "J1") (unit 1) (value "Conn_01x05") (footprint "Molex-53015:Molex_MicroBlade_53015-0500_1x05_P2.00mm_Right")
+      (reference "J1") (unit 1) (value "53015-0510") (footprint "Molex-53015:Molex_MicroBlade_53015-0500_1x05_P2.00mm_Right")
     )
     (path "/93d9434f-baa4-45e9-b1ac-4fbddd6d48ca/40515802-9162-43b0-b44b-636b1b77036c"
-      (reference "J2") (unit 1) (value "53014-1010") (footprint "Molex-53015:Molex_MicroBlade_53015-1000_1x10_P2.00mm_Right")
+      (reference "J2") (unit 1) (value "53015-0510") (footprint "Molex-53015:Molex_MicroBlade_53015-1000_1x10_P2.00mm_Right")
     )
     (path "/6dfaa3f9-076c-470d-9afe-3e64c474240c/4d251ecf-72e4-433c-9336-46d24256d8e2"
@@
     )
     (path "/6dfaa3f9-076c-470d-9afe-3e64c474240c/eacf09c8-8283-40fb-a003-cb9032cd9787"
-      (reference "L2") (unit 1) (value "MCF-1040-330-N2") (footprint "Inductor_SMD:L_12x12mm_H6mm")
+      (reference "L2") (unit 1) (value "MWSA1206S-330MT") (footprint "Power_Inductor_Extended:L_Sunlord-MWSA1206S")
     )
     (path "/93d9434f-baa4-45e9-b1ac-4fbddd6d48ca/ee10f824-29d5-44db-88cf-610f4ef786cc"
@@
       (reference "R17") (unit 1) (value "1.13k") (footprint "Resistor_SMD:R_0603_1608Metric")
     )
+    (path "/d8acfe39-023f-4fd0-8eb6-48564869a83e"
+      (reference "SYM1") (unit 1) (value "SYM_Arrow_Tiny") (footprint "Symbol_Extended:LamudaEE-12.8x7.9mm")
+    )
     (path "/fbae0290-fe5d-40de-8e10-f5a0736b65f7"

Commit message: update bom2
Parts:
- DEBUG1: Supplier N/C -> (none)
- SYM1, TP1: Mount (none) -> N/C
- U1: LCSC Part (none) -> C529330; MFR.Part# (none) -> STM32G030F6P6TR; Manufacturer (none) -> STMicroelectronics; Mount (none) -> SMD; ODR.Part# (none) -> STM32G030F6P6TR; Packaging (none) -> TSSOP-20; Supplier (none) -> JLCPCB-Extended
Changed lines of the file:
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@@
+      (effects (font (size 1.27 1.27)) hide)
+    )
+    (property "Mount" "N/C" (id 4) (at 213.36 124.46 0)
       (effects (font (size 1.27 1.27)) hide)
     )
@@
       (effects (font (size 1.27 1.27)) hide)
     )
+    (property "Mount" "N/C" (id 4) (at 154.94 97.79 0)
+      (effects (font (size 1.27 1.27)) hide)
+    )
     (pin "1")
   )
@@
       (effects (font (size 1.27 1.27)) hide)
     )
-    (property "Supplier" "N/C" (id 5) (at 93.98 76.2 0)
+    (property "Supplier" "" (id 5) (at 93.98 76.2 0)
       (effects (font (size 1.27 1.27)) hide)
     )
@@
       (effects (font (size 1.27 1.27)) hide)
     )
+    (property "LCSC Part" "C529330" (id 4) (at 96.52 46.99 0)
+      (effects (font (size 1.27 1.27)) hide)
+    )
+    (property "MFR.Part#" "STM32G030F6P6TR" (id 5) (at 96.52 46.99 0)
+      (effects (font (size 1.27 1.27)) hide)
+    )
+    (property "Manufacturer" "STMicroelectronics" (id 6) (at 96.52 46.99 0)
+      (effects (font (size 1.27 1.27)) hide)
+    )
+    (property "Mount" "SMD" (id 7) (at 96.52 46.99 0)
+      (effects (font (size 1.27 1.27)) hide)
+    )
+    (property "ODR.Part#" "STM32G030F6P6TR" (id 8) (at 96.52 46.99 0)
+      (effects (font (size 1.27 1.27)) hide)
+    )
+    (property "Packaging" "TSSOP-20" (id 9) (at 96.52 46.99 0)
+      (effects (font (size 1.27 1.27)) hide)
+    )
+    (property "Supplier" "JLCPCB-Extended" (id 10) (at 96.52 46.99 0)
+      (effects (font (size 1.27 1.27)) hide)
+    )

Commit message: updates pdf.
Other:
- company: (none) -> Korean Paper Dispenser Parallel to Serial Module
- title: (none) -> Main Block
Changed lines of the file:
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@@
 (kicad_sch (version 20210621) (generator eeschema)
   (paper "A4")
+  (title_block
+    (title "Main Block")
+    (date "2021-07-30")
+    (rev "0.1")
+    (company "Korean Paper Dispenser Parallel to Serial Module")
+    (comment 1 "Features : 24V -> 12V, RS232, STM32G030")
+    (comment 2 "Proof of concept hardware for Rust-Embedded.")
+    (comment 3 "CERN-OHL-S-2.0")
+    (comment 4 "Jinwoo Park pmnxis@gmail.com")
+  )
   (junction (at 39.37 33.02) (diameter 0.9144) (color 0 0 0 0))
   (junction (at 39.37 40.64) (diameter 0.9144) (color 0 0 0 0))

Commit message: pre 2
Parts:
- added D3: SMBJ28CA, Diode_SMD:D_SMB, symbol Device:D_TVS
- added SYM2: SYM_Arrow_Tiny, Symbol:OSHW-Logo2_14.6x12mm_SilkScreen, symbol Graphic:SYM_Arrow_Tiny
- D1, D2: value LED GREEN -> LED_YELLOW; LCSC Part C2297 -> C2296; MFR.Part# KT-0805G -> KT-0805Y; ODR.Part# LED GREEN 2012 -> LED YELLOW 2012
Connections:
- net +24V: now also D3.2 (A2)
- net GND: now also D3.1 (A1)
Other:
- note added: "github.com/PapoutPSM-HW.git"
- company: Korean Paper Dispenser Parallel to Serial Module -> Korean Paper Dispenser Parallel to Serial Adapter Module

Commit message: release/v3 update
Parts:
- C1: LCSC Part C1525 -> C23733; MFR.Part# CL05B104KO5NNNC -> CL05A475MP5NRNC
- U1: value STM32G030F6 -> STM32G031F8P6; LCSC Part C529330 -> C529334; MFR.Part# STM32G030F6P6TR -> STM32G031F8P6; ODR.Part# STM32G030F6P6TR -> STM32G031F8P6
Connections:
- net P_EMPTY: now also U1.15 (PB0/PB1/PB2/PA8); no longer U1.12 (PA5)
- net P_ERROR: now also U1.16 (PA11_[PA9]); no longer U1.11 (PA4)
- net P_INHIBIT: now also U1.11 (PA4); no longer U1.16 (PA11_[PA9])
- net P_OUT_PULSE: now also U1.14 (PA7); no longer U1.13 (PA6)
- net P_PULSE: now also U1.13 (PA6); no longer U1.14 (PA7)
- net P_RESET: now also U1.12 (PA5); no longer U1.15 (PB0/PB1/PB2/PA8)
