File: PapoutPSM-HW.kicad_sch (KiCad schematic)
At the start: 24 parts, among them J1 53015-0510, U1 STM32G031F8P6, U2 SP3232EEY-L

Commit message: before release v0.5
Parts:
- removed C8: 100nF, Capacitor_SMD:C_0402_1005Metric, symbol Device:C
- removed D1, D2: LED_YELLOW, LED_SMD:LED_0805_2012Metric, symbol Device:LED
- removed D3: SMBJ28CA, Diode_SMD:D_SMB, symbol Device:D_TVS
- removed DEBUG1: TC2030-IDC, Connector:Tag-Connect_TC2030-IDC-FP_2x03_P1.27mm_Vertical, symbol Connector_Generic:Conn_02x03_Odd_Even
- removed J1: 53015-0510, Molex-53015:Molex_MicroBlade_53015-0500_1x05_P2.00mm_Right, symbol Connector_Generic:Conn_01x05
- removed TP1: TestPoint, TestPoint:TestPoint_Pad_D1.0mm, symbol Connector:TestPoint
- removed U1: STM32G031F8P6, Package_SO:TSSOP-20_4.4x6.5mm_P0.65mm, symbol STM32G0:STM32G030F6
- removed U2: SP3232EEY-L, Package_SO:TSSOP-16_4.4x5mm_P0.65mm, symbol Interface_UART_Extended:SP3232EEY-L
- added C10: 100nF 50V, Capacitor_SMD:C_0603_1608Metric, symbol Device:C
- added C11, C8, C9: 1.8mF, Capacitor_THT:CP_Radial_D12.5mm_P5.00mm, symbol Device:C_Polarized
- added C12, C18, C23, C25, C26, C27, C28: 100nF, Capacitor_SMD:C_0402_1005Metric, symbol Device:C
- added C13, C14: 47uF, Capacitor_SMD:C_1210_3225Metric, symbol Device:C
- added C15, C16, C17, C20, C21, C22: 100nF, Capacitor_SMD:C_0402_1005Metric, symbol Device:C_Small
- added C19: 10uF 50V, Capacitor_SMD:C_0805_2012Metric, symbol Device:C
- added C24: 1nF, Capacitor_SMD:C_0402_1005Metric, symbol Device:C
- added D1: 1N4007, Diode_THT:D_DO-41_SOD81_P10.16mm_Horizontal, symbol Diode:1N4007
- added D10, D11, D12, D4, D5, D6: 1N4007, Diode_SMD:D_SOD-123F, symbol Diode:1N4007
- added D13: SMBJ28CA, Diode_SMD:D_SMB, symbol Device:D_TVS
- added D2: 1N4148W, Diode_SMD:D_SOD-123, symbol Diode:1N4148W
- added D3: SS34, Diode_SMD:D_SMA, symbol Device:D_Schottky
- added D7, D8: LED_YELLOW, LED_SMD:LED_0805_2012Metric, symbol Device:LED
- added D9: LED GREEN, LED_SMD:LED_0805_2012Metric, symbol Device:LED
- added DEBUG1: TC2030-IDC, Connector:Tag-Connect_TC2030-IDC-FP_2x03_P1.27mm_Vertical, symbol Connector_Generic:Conn_02x03_Counter_Clockwise
- added FB1, FB2, FB3, FB4, FB5, FB6: GZ2012D601TF, Inductor_SMD:L_0805_2012Metric, symbol Device:FerriteBead_Small
- added J1: 53015-0510, Molex-53015:Molex_MicroBlade_53015-1000_1x10_P2.00mm_Right, symbol Connector_Generic:Conn_01x10
- added J2: Barrel_Jack, Connector_BarrelJack:BarrelJack_GCT_DCJ200-10-A_Horizontal, symbol Connector:Barrel_Jack_Switch_Pin3Ring
- added J3: 53015-0510, Molex-53015:Molex_MicroBlade_53015-0500_1x05_P2.00mm_Right, symbol Connector_Generic:Conn_01x05
- added L1: FNR6045S222KT, Inductor_SMD:L_Bourns_SRN6045TA, symbol Power_Inductor_Extended:NR6028T4R7M
- added L2: CDRH8D43NP-6R8NC, Inductor_SMD:L_Bourns-SRU8028_8.0x8.0mm, symbol Power_Inductor_Extended:NR6028T4R7M
- added Q1, Q2, Q3: 2N7002, Package_TO_SOT_SMD:SOT-23, symbol Transistor_FET:2N7002
- added R10, R11, R14, R15, R16, R18, R20, R22, R4, R5, R6: 4.7k, Resistor_SMD:R_0402_1005Metric, symbol Device:R_US
- added R12: 10k, Resistor_SMD:R_0402_1005Metric, symbol Device:R_US
- added R13: 47k, Resistor_SMD:R_0402_1005Metric, symbol Device:R_US
- added R17, R19, R21: 660, Resistor_SMD:R_0603_1608Metric, symbol Device:R_US
- added R3: 12k, Resistor_SMD:R_0603_1608Metric, symbol Device:R_US
- added R7, R8, R9: 330, Resistor_SMD:R_0603_1608Metric, symbol Device:R_US
- added RV1: 10Ø 18V, Varistor:RV_Disc_D12mm_W4.3mm_P7.5mm, symbol Device:Varistor
- added SW1: DSIC04LSGET, Button_Switch_SMD_Extended:SW_DIP_SPSTx04_Slide_9.30x10.16mm_W4.25mm_P2.54mm, symbol Switch:SW_DIP_x04
- added U1: LMR14020SDDA, Package_SO:TI_SO-PowerPAD-8_ThermalVias, symbol Regulator_Switching_Extended:LMR14050SDDA
- added U10: SP3232EEY-L, Package_SO:TSSOP-16_4.4x5mm_P0.65mm, symbol Interface_UART_Extended:SP3232EEY-L
- added U2: 78L05G-AB3-R, Package_TO_SOT_SMD:SOT-89-3, symbol Regulator_Linear:NCP1117-5.0_TO252
- added U3, U4, U5, U6, U7, U8: EL3H7-G, EL3H7-G:SMDIP-4_W5.20mm, symbol Isolator:LTV-817S
- added U9: MSP430FR2433IRGE, Package_DFN_QFN:HVQFN-24-1EP_4x4mm_P0.5mm_EP2.5x2.5mm, symbol MSP430FR2433:MSP430FR2433IRGE
- C1: value 4.7uF -> 10uF 50V; footprint Capacitor_SMD:C_0402_1005Metric -> Capacitor_SMD:C_0805_2012Metric; LCSC Part C23733 -> C440198; MFR.Part# CL05A475MP5NRNC -> GRM21BR61H106KE43L; Manufacturer ANY -> Murata; ODR.Part# CAP 100nF 1005 -> CAP 10uF 50V 2012; Packaging 1005 -> 2012
- C2, C7: value 100nF -> 330nF; footprint Capacitor_SMD:C_0402_1005Metric -> Capacitor_SMD:C_0805_2012Metric; LCSC Part C1525 -> C1740; MFR.Part# CL05B104KO5NNNC -> 0805B334K500NT; ODR.Part# CAP 100nF 1005 -> CAP 330nF 2012; Packaging 1005 -> 2012
- C3: LCSC Part C1525 -> C307331; MFR.Part# CL05B104KO5NNNC -> CL05B104KB54PNC
- C4: value 100nF -> 220pF; footprint Capacitor_SMD:C_0402_1005Metric -> Capacitor_SMD:C_0603_1608Metric; LCSC Part C1525 -> C1664; MFR.Part# CL05B104KO5NNNC -> CL10C331JB8NNNC; ODR.Part# CAP 100nF 1005 -> CAP 330pF 1608; Packaging 1005 -> 1608
- C5: value 100nF -> 22nF; footprint Capacitor_SMD:C_0402_1005Metric -> Capacitor_SMD:C_0603_1608Metric; LCSC Part C1525 -> C21122; MFR.Part# CL05B104KO5NNNC -> CL10B223KB8NNNC; ODR.Part# CAP 100nF 1005 -> CAP 22nF 1608; Packaging 1005 -> 1608
- C6: value 100nF -> 1uF; footprint Capacitor_SMD:C_0402_1005Metric -> Capacitor_THT:C_Rect_L7.5mm_W6.5mm_P5.00mm; LCSC Part C1525 -> (none); MFR.Part# CL05B104KO5NNNC -> MMY105J100V; ODR.Part# CAP 100nF 1005 -> CBB 1uF; Supplier JLCPCB-Basic -> Hand-Soldering
- R1: value 4.7k -> 20k; footprint Resistor_SMD:R_0402_1005Metric -> Resistor_SMD:R_0603_1608Metric; LCSC Part C25900 -> C4184; MFR.Part# 0402WGF4701TCE -> 0603WAF2002T5E; ODR.Part# RES 4.7k 1005 -> RES 20k 1% 1608; Packaging 1005 -> 1608
- R2: value 4.7k -> 68k; footprint Resistor_SMD:R_0402_1005Metric -> Resistor_SMD:R_0603_1608Metric; LCSC Part C25900 -> C22807; MFR.Part# 0402WGF4701TCE -> 0603WAF1503T5E; ODR.Part# RES 4.7k 1005 -> RES 150k 1% 1608; Packaging 1005 -> 1608
Connections:
- net +24V: now also C1.1, C3.1, D13.2 (A2), J3.1 (Pin_1), U1.2 (VIN), U1.3 (EN)
- net +3V3: now also R2.1, C13.1, C14.1, C18.1, C19.1, C23.1, D10.2 (A), D11.2 (A), D12.2 (A), DEBUG1.6 (Pin_6), L2.2, R12.1, R13.2, R17.2, R19.2, R21.2, U10.16 (VCC), U9.24 (DVCC); no longer C1.1, C3.1, C7.2
- net GND: now also C5.2, R1.2, C13.2, C14.2, C18.2, C19.2, C20.2, C21.2, C22.2, C23.2, C24.2, C27.1, C28.1, D13.1 (A1), D3.2 (A), D7.1 (K), D8.1 (K), D9.1 (K), DEBUG1.4 (Pin_4), J3.2 (Pin_2), J3.3 (Pin_3), R3.2, SW1.5, SW1.6, SW1.7, SW1.8, U1.7 (GND), U1.9 (EP), U10.10 (T2IN), U10.15 (GND), U10.8 (R2IN), U3.2, U4.2, U5.2, U6.3, U7.3, U8.3, U9.18 (DVSS), U9.20 (P3.2), U9.21 (P2.0/XIN), U9.22 (P2.1/XOUT), U9.23 (DVSS), U9.25 (EP); no longer C2.2, C4.2
- net LED0: now also R10.1, U9.15 (UCA1CLK/P2.4); no longer R1.1
- net LED1: now also R11.1, U9.19 (P2.7); no longer R2.1
- net M_RX: now also U10.14 (T1OUT), U9.16 (UCA1SOMI_/UCA1RXD/P2.5)
- net M_TX: now also U10.13 (R1IN), U9.17 (UCA1SIMO/UCA1TXD/P2.6)
- net NRST: now also C24.1, DEBUG1.5 (Pin_5), R13.1, U9.1 (~{RST}/NMI/SBWTDIO); no longer C2.1
- net P_EMPTY: now also C21.1, R15.2, U7.4, U9.13 (P2.3)
- net P_ERROR: now also C22.1, R16.2, U8.4, U9.14 (UCA1STE/P3.1)
- net P_INHIBIT: now also R18.2, U9.9 (TA0.2/Veref-/UCB0SDA/UCB0SIMO/A2/P1.2)
- net P_OUT_PULSE: now also C20.1, R14.2, U6.4, U9.12 (P3.0)
- net P_PULSE: now also R22.2, U9.11 (ACLK/P2.2)
- net P_RESET: now also R20.2, U9.10 (MCLK/UCB0SCL/UCB0SOMI/A3/P1.3)
- net R_RXD: now also J3.5 (Pin_5), U10.12 (R1OUT)
- net R_TXD: now also J3.4 (Pin_4), U10.11 (T1IN)
- net BIG_FB: now reaches R2.2
- net BIG_FB: now also C4.2, R3.1, U1.5 (FB)
- net BIG_SS: now reaches C5.1
- net BIG_SS: now also U1.6 (SS)
- net +FILTERED_12VA: now reaches C7.1
- net +FILTERED_12VA: now also D2.1 (K), L1.2, U2.3 (VI)
- net GNDA: now reaches C6.2
- net GNDA: now also C2.2, C7.2, C11.2, C12.2, C15.1, C16.1, C17.1, C8.2, C9.2, D1.2 (A), J1.10 (Pin_10), J1.9 (Pin_9), J2.2, J2.3, RV1.2, U2.1 (GND), U3.3, U4.3, U5.3, U6.2, U7.2, U8.2
- net +12VA: now reaches C6.1
- net +12VA: now also C2.1, C11.1, C8.1, C9.1, D1.1 (K), J1.7 (Pin_7), J1.8 (Pin_8), J2.1, L1.1, RV1.1
- new net: D12.1 (K), R16.1
- new net: D8.2 (A), R11.2
- new net: Q3.1 (G), R22.1
- new net: D9.2 (A), R12.2
- new net: Q2.1 (G), R20.1
- new net: Q2.3 (D), R19.1
- new net: D6.1 (K), R6.1
- new net: Q3.3 (D), R21.1
- new net: C25.2, U10.1 (C1+)
- new net: C27.2, U10.2 (V+)
- new net: C25.1, U10.3 (C1-)
- new net: C26.2, U10.4 (C2+)
- new net: C26.1, U10.5 (C2-)
- new net: C28.2, U10.6 (V-)
- new net: D11.1 (K), R15.1
- new net: D7.2 (A), R10.2
- new net: Q1.1 (G), R18.1
- new net: Q1.3 (D), R17.1
- new net: D10.1 (K), R14.1
- new net: D5.1 (K), R5.1
- new net: D4.1 (K), R4.1
- new net +5VA: C12.1, D2.2 (A), D4.2 (A), D5.2 (A), D6.2 (A), U2.2 (VO)
- new net ANODE_EMPTY: R8.2, U7.1
- new net ANODE_ERROR: R9.2, U8.1
- new net ANODE_INHIBIT: Q1.2 (S), U3.1
- new net ANODE_OUT_PULSE: R7.2, U6.1
- new net ANODE_PULSE: Q3.2 (S), U5.1
- new net ANODE_RESET: Q2.2 (S), U4.1
- new net BIG_BOOT: C10.1, U1.1 (BOOT)
- new net BIG_RTS: R1.1, U1.4 (RT/SYNC)
- new net BIG_SW: C10.2, D3.1 (K), L2.1, U1.8 (SW)
- new net D_RX: DEBUG1.2 (Pin_2), U9.4 (P1.5/TMS/UCA0SOMI/UCA0RXD/A5/TA1.1)
- new net D_TX: DEBUG1.1 (Pin_1), U9.3 (P1.4/TCK/VREF+/UCA0SIMO/UCA0TXD/A4/TA1.2)
- new net EX_EMPTY: FB5.1, J1.5 (Pin_5)
- new net EX_ERROR: FB6.1, J1.6 (Pin_6)
- new net EX_INHIBIT: FB1.1, J1.1 (Pin_1)
- new net EX_OUT_PULSE: FB4.1, J1.4 (Pin_4)
- new net EX_PULSE: FB3.1, J1.3 (Pin_3)
- new net EX_RESET: FB2.1, J1.2 (Pin_2)
- new net J_EMPTY: FB5.2, R8.1
- new net J_ERROR: FB6.2, R9.1
- new net J_INHIBIT: C17.2, FB1.2, R4.2, U3.4
- new net J_OUT_PULSE: FB4.2, R7.1
- new net J_PULSE: C16.2, FB3.2, R6.2, U5.4
- new net J_RESET: C15.2, FB2.2, R5.2, U4.4
- new net SW0: SW1.1, U9.8 (TA0.1/A1/UCB0CLK/A0/P1.1)
- new net SW1: SW1.2, U9.5 (P1.6/TDI/TCLK/TA1CLK/UCA0CLK/A6)
- new net SW2: SW1.3, U9.6 (P1.7/TDO/UCA0STE/SMCLK/A7)
- new net SW3: SW1.4, U9.7 (TA0CLK/Veref+/UCB0STE/A0/P1.0)
- new net TEST: DEBUG1.3 (Pin_3), U9.2 (TEST/SBWTCK)
- no-connect marks 3 -> 2
Other:
- removed sheet Parallel_IO
- removed sheet Power
- note added: "1000uF ~ 1200uF 25~35V ESR <= 50mΩ@100Khz I(Ripple) >= 2.0A@100Khz"
- note added: "Alter B340"
- note added: "ISOLATION"
- note added: "ISOLATION - MOTOR SIDE"
- note added: "Large Thermal"
- note added: "Motor (Paper Dispenser Side)"
- note added: "Motor Noise Filter Noise = 10Mhz (Vgap 1-4V) 1mH <="
- note added: "Original pin map start with 1 from here"
- note added: "Regulator and MCU Side"
- note added: "Soft Start 5msecs"
- note added: "TODO:Change to LowSide"
- note added: "Varistor should be replaced when use for 24V"
- note removed: "github.com/PapoutPSM-HW.git"
- company: Korean Paper Dispenser Parallel to Serial Adapter Module -> Jinwoo Park (pmnxis@gmail.com)
- title: Main Block -> PapoutPSM-HW
