File: PapoutPSM-HW.kicad_sch (KiCad schematic)
At the start: 96 parts, among them J1 53015-0510, J2 Barrel_Jack, J3 53015-0510, Q1 2N7002, Q2 2N7002, Q3 2N7002, SW1 DSIC04LSGET, U1 LMR14020SDDA, U10 SP3232EEY-L, U2 78L05G-AB3-R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

Commit message: Update latest changes on low-side NMos usage
Connections:
- net ANODE_INHIBIT: now also R17.1; no longer Q1.2 (S)
- net ANODE_PULSE: now also R21.1; no longer Q3.2 (S)
- net ANODE_RESET: now also R19.1; no longer Q2.2 (S)
- net GND: now also Q1.2 (S), Q2.2 (S), Q3.2 (S); no longer U3.2, U4.2, U5.2
- net CATHODE_RESET: now reaches Q2.3 (D)
- net CATHODE_RESET: now also U4.2; no longer R19.1
- net CATHODE_PULSE: now reaches Q3.3 (D)
- net CATHODE_PULSE: now also U5.2; no longer R21.1
- net CATHODE_INHIBIT: now reaches Q1.3 (D)
- net CATHODE_INHIBIT: now also U3.2; no longer R17.1
Other:
- moved on the sheet: Q1, Q2, Q3, R17, R18, R19, R20, R21, R22
