File: Parallel_IO.kicad_sch (KiCad schematic)
At the start: 50 parts, among them J2 53015-0510, U3 LTV-817S, U4 LTV-817S, U5 LTV-817S, U6 LTV-817S, U7 LTV-817S, U8 LTV-817S

Commit message: some layout changed (sizeup for later 2layer conversion)
Parts:
- renumbered C9 to C10, C10 to C11, C11 to C12, C12 to C13, C13 to C14, C14 to C15, C15 to C16, C16 to C17, C17 to C18, C18 to C19, C19 to C20, C20 to C21, C21 to C22, U3 to U4, U4 to U5, U5 to U6, U6 to U7, U7 to U8, U8 to U9
Changed lines of the file:
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@@
   (symbol (lib_id "Device:C") (at 39.37 57.15 0) (unit 1)
     (in_bom yes) (on_board yes)
-    (property "Reference" "C9" (id 0) (at 41.91 55.88 0)
+    (property "Reference" "C10" (id 0) (at 41.91 55.88 0)
       (effects (font (size 1.27 1.27)) (justify left))
     )
@@
   (symbol (lib_id "Device:C") (at 39.37 104.14 0) (unit 1)
     (in_bom yes) (on_board yes)
-    (property "Reference" "C10" (id 0) (at 41.91 102.87 0)
+    (property "Reference" "C11" (id 0) (at 41.91 102.87 0)
       (effects (font (size 1.27 1.27)) (justify left))
     )
@@
   (symbol (lib_id "Device:C") (at 39.37 151.13 0) (unit 1)
     (in_bom yes) (on_board yes)
-    (property "Reference" "C11" (id 0) (at 41.91 149.86 0)
+    (property "Reference" "C12" (id 0) (at 41.91 149.86 0)
       (effects (font (size 1.27 1.27)) (justify left))
     )
@@
   (symbol (lib_id "Device:C") (at 118.11 57.15 0) (unit 1)
     (in_bom yes) (on_board yes)
-    (property "Reference" "C12" (id 0) (at 120.65 55.88 0)
+    (property "Reference" "C13" (id 0) (at 120.65 55.88 0)
       (effects (font (size 1.27 1.27)) (justify left))
     )
@@
   (symbol (lib_id "Device:C") (at 118.11 104.14 0) (unit 1)
     (in_bom yes) (on_board yes)
-    (property "Reference" "C13" (id 0) (at 120.65 102.87 0)
+    (property "Reference" "C14" (id 0) (at 120.65 102.87 0)
       (effects (font (size 1.27 1.27)) (justify left))
     )
@@
   (symbol (lib_id "Device:C") (at 118.11 151.13 0) (unit 1)
     (in_bom yes) (on_board yes)
-    (property "Reference" "C14" (id 0) (at 120.65 149.86 0)
+    (property "Reference" "C15" (id 0) (at 120.65 149.86 0)
       (effects (font (size 1.27 1.27)) (justify left))
     )
@@
   (symbol (lib_id "Device:C") (at 149.86 57.15 0) (unit 1)
     (in_bom yes) (on_board yes)
-    (property "Reference" "C15" (id 0) (at 152.4 55.88 0)
+    (property "Reference" "C16" (id 0) (at 152.4 55.88 0)
       (effects (font (size 1.27 1.27)) (justify left))
     )
@@
   (symbol (lib_id "Device:C") (at 149.86 104.14 0) (unit 1)
     (in_bom yes) (on_board yes)
-    (property "Reference" "C16" (id 0) (at 152.4 102.87 0)
+    (property "Reference" "C17" (id 0) (at 152.4 102.87 0)
       (effects (font (size 1.27 1.27)) (justify left))
     )
@@
   (symbol (lib_id "Device:C") (at 149.86 151.13 0) (unit 1)
     (in_bom yes) (on_board yes)
-    (property "Reference" "C17" (id 0) (at 152.4 149.86 0)
+    (property "Reference" "C18" (id 0) (at 152.4 149.86 0)
       (effects (font (size 1.27 1.27)) (justify left))
     )
@@
   (symbol (lib_id "Device:C") (at 199.39 151.13 0) (mirror y) (unit 1)
     (in_bom yes) (on_board yes)
-    (property "Reference" "C18" (id 0) (at 201.93 149.8599 0)
+    (property "Reference" "C19" (id 0) (at 201.93 149.8599 0)
       (effects (font (size 1.27 1.27)) (justify right))
     )
@@
   (symbol (lib_id "Device:C_Polarized") (at 232.41 151.13 0) (unit 1)
     (in_bom yes) (on_board yes)
-    (property "Reference" "C19" (id 0) (at 234.95 149.8599 0)
+    (property "Reference" "C20" (id 0) (at 234.95 149.8599 0)
       (effects (font (size 1.27 1.27)) (justify left))
     )
@@
   (symbol (lib_id "Device:C_Polarized") (at 242.57 151.13 0) (unit 1)
     (in_bom yes) (on_board yes)
-    (property "Reference" "C20" (id 0) (at 245.11 149.8599 0)
+    (property "Reference" "C21" (id 0) (at 245.11 149.8599 0)
       (effects (font (size 1.27 1.27)) (justify left))
     )
@@
   (symbol (lib_id "Device:C_Polarized") (at 252.73 151.13 0) (unit 1)
     (in_bom yes) (on_board yes)
-    (property "Reference" "C21" (id 0) (at 255.27 149.8599 0)
+    (property "Reference" "C22" (id 0) (at 255.27 149.8599 0)
       (effects (font (size 1.27 1.27)) (justify left))
     )
@@
   (symbol (lib_id "Isolator:LTV-817S") (at 57.15 54.61 0) (unit 1)
     (in_bom yes) (on_board yes) (fields_autoplaced)
-    (property "Reference" "U3" (id 0) (at 57.15 45.72 0))
+    (property "Reference" "U4" (id 0) (at 57.15 45.72 0))
     (property "Value" "LTV-817S" (id 1) (at 57.15 48.26 0))
     (property "Footprint" "Package_DIP:SMDIP-4_W9.53mm" (id 2) (at 57.15 62.23 0)
@@
   (symbol (lib_id "Isolator:LTV-817S") (at 57.15 101.6 0) (unit 1)
     (in_bom yes) (on_board yes) (fields_autoplaced)
-    (property "Reference" "U4" (id 0) (at 57.15 92.71 0))
+    (property "Reference" "U5" (id 0) (at 57.15 92.71 0))
     (property "Value" "LTV-817S" (id 1) (at 57.15 95.25 0))
     (property "Footprint" "Package_DIP:SMDIP-4_W9.53mm" (id 2) (at 57.15 109.22 0)
@@
   (symbol (lib_id "Isolator:LTV-817S") (at 57.15 148.59 0) (unit 1)
     (in_bom yes) (on_board yes) (fields_autoplaced)
-    (property "Reference" "U5" (id 0) (at 57.15 139.7 0))
+    (property "Reference" "U6" (id 0) (at 57.15 139.7 0))
     (property "Value" "LTV-817S" (id 1) (at 57.15 142.24 0))
     (property "Footprint" "Package_DIP:SMDIP-4_W9.53mm" (id 2) (at 57.15 156.21 0)
@@
   (symbol (lib_id "Isolator:LTV-817S") (at 135.89 54.61 0) (unit 1)
     (in_bom yes) (on_board yes) (fields_autoplaced)
-    (property "Reference" "U6" (id 0) (at 135.89 45.72 0))
+    (property "Reference" "U7" (id 0) (at 135.89 45.72 0))
     (property "Value" "LTV-817S" (id 1) (at 135.89 48.26 0))
     (property "Footprint" "Package_DIP:SMDIP-4_W9.53mm" (id 2) (at 135.89 62.23 0)
@@
   (symbol (lib_id "Isolator:LTV-817S") (at 135.89 101.6 0) (unit 1)
     (in_bom yes) (on_board yes) (fields_autoplaced)
-    (property "Reference" "U7" (id 0) (at 135.89 92.71 0))
+    (property "Reference" "U8" (id 0) (at 135.89 92.71 0))
     (property "Value" "LTV-817S" (id 1) (at 135.89 95.25 0))
     (property "Footprint" "Package_DIP:SMDIP-4_W9.53mm" (id 2) (at 135.89 109.22 0)
@@
   (symbol (lib_id "Isolator:LTV-817S") (at 135.89 148.59 0) (unit 1)
     (in_bom yes) (on_board yes) (fields_autoplaced)
-    (property "Reference" "U8" (id 0) (at 135.89 139.7 0))
+    (property "Reference" "U9" (id 0) (at 135.89 139.7 0))
     (property "Value" "LTV-817S" (id 1) (at 135.89 142.24 0))
     (property "Footprint" "Package_DIP:SMDIP-4_W9.53mm" (id 2) (at 135.89 156.21 0)
