File: Parallel_IO.kicad_sch (KiCad schematic)
At the start: 26 parts, among them Q1 NTK3134NT1G, Q2 NTK3134NT1G, U1 74HC4049

Commit message: v1
Parts:
- removed C10, C11: 100nF, Capacitor_SMD:C_0402_1005Metric, symbol Device:C
- removed C12, C15: 22uF, Capacitor_SMD:C_0805_2012Metric, symbol Device:C
- removed C13, C14, C8: 10nF, Capacitor_SMD:C_0402_1005Metric, symbol Device:C
- removed R13: 4.7k, Resistor_SMD:R_0402_1005Metric, symbol Device:R_US
- removed R17, R20, R21: 51k, Resistor_SMD:R_0402_1005Metric, symbol Device:R_US
- added J2: 53014-1010, Molex-53015:Molex_MicroBlade_53015-1000_1x10_P2.00mm_Right, symbol Connector_Generic:Conn_01x10
- added Q3: NTK3134NT1G, Package_TO_SOT_SMD:SOT-723, symbol Transistor_FET_Extended:DMN100-7-F
- added R5: 4.7k, Resistor_SMD:R_0402_1005Metric, symbol Device:R_US
- U3: renamed from U1; footprint Package_SO:TSSOP-16_4.4x5mm_P0.65mm -> Package_SO:SOIC-16_3.9x9.9mm_P1.27mm
- renumbered C6 to C10, C7 to C11, C9 to C12, C5 to C9, R15 to R10, R16 to R11, R18 to R3, R19 to R4, R10 to R6, R11 to R7, R12 to R8, R14 to R9
Connections:
- net +12V: now also J2.3 (Pin_3), J2.4 (Pin_4), R5.2
- net GND: now also U3.3, U3.5, U3.7, J2.1 (Pin_1), J2.2 (Pin_2), Q3.2 (S)
- net at U3.14: now also C9.1, R9.2
- net at C11.1, R11.2: now also U3.9; no longer U3.5
- net at U3.11: now also C10.1, R10.2
- net FE_VVIN0 renamed J_OUT_PULSE
- net J_OUT_PULSE: now also J2.7 (Pin_7)
- net FE_VVIN1 renamed J_EMPTY
- net J_EMPTY: now also J2.6 (Pin_6)
- net FE_VVIN2 renamed J_ERROR
- net J_ERROR: now also J2.5 (Pin_5)
- net FE_VVOU0 renamed J_INHIBIT
- net J_INHIBIT: now also J2.10 (Pin_10)
- net FE_VVOU1 renamed J_RESET
- net J_RESET: now also J2.9 (Pin_9)
- net PCIN0 renamed P_EMPTY
- net PCIN1 renamed P_OUT_PULSE
- net VVIN0 renamed P_ERROR
- net VVIN1: no longer names the net of U3.6
- net VVIN2: no longer names the net of U3.4
- net VVIN3: no longer names the net of U3.2
- net VVOU0 renamed P_INHIBIT
- net VVOU1 renamed P_RESET
- new net J_PULSE: J2.8 (Pin_8), Q3.3 (D), R5.1
- new net P_PULSE: Q3.1 (G)
- no-connect marks 0 -> 3
Other:
- note added: "NOT-USE"
- note added: "VEND Open Drain 2"
- note removed: "2020-07-16 : LTV217 Optocopuler is removed. Replaced to high voltage input hex inverter. Ti CD4049UBDR recommend 1uA input. Ti require too few input current. So this design use "ONSemi MC14049UBDR2G" , "Nxp HEF4049BT""
- note removed: "2020-07-20 : DMN100 or PMV100 NMOS reduce to dual channel NMOS. DMN3190LDW or DMN2004DWK Recommend is DMN3190LDW , Alternative is DMN2004DWK Requirements : high desity, high current and voltage accept. Gate,D-S Protection."
- note removed: "2020-07-20 : DMN100 or PMV100 NMOS reduce to dual channel NMOS. Recommend is DMN3190LDW and Alternative is DMN2004DWK Requirements : high desity, high current , Volt accept. Gate,D-S Protection."
- note removed: "CHANGE LOG"
- note removed: "PCB Side extSignal Invert Input"
- note removed: "PCB Sig Invert 0"
- note removed: "PCB Sig Invert 1"
- note removed: "VEND Pull Up 3"
- moved on the sheet: C10, C11, C12, C9, Q1, Q2, R10, R11, R3, R4, R6, R7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

Commit message: update bom
Parts:
- J2: value 53014-1010 -> 53015-0510; MFR.Part# 53014-1010 -> 53015-1010; ODR.Part# 53014-1010 -> 53015-1010
Changed lines of the file:
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@@
       (effects (font (size 1.27 1.27)) (justify left))
     )
-    (property "Value" "53014-1010" (id 1) (at 266.7 158.75 0)
+    (property "Value" "53015-0510" (id 1) (at 266.7 158.75 0)
       (effects (font (size 1.27 1.27)) (justify left))
     )
@@
       (effects (font (size 1.27 1.27)) hide)
     )
-    (property "MFR.Part#" "53014-1010" (id 4) (at 271.78 144.78 0)
+    (property "MFR.Part#" "53015-1010" (id 4) (at 271.78 144.78 0)
       (effects (font (size 1.27 1.27)) hide)
     )
@@
       (effects (font (size 1.27 1.27)) hide)
     )
-    (property "ODR.Part#" "53014-1010" (id 7) (at 271.78 144.78 0)
+    (property "ODR.Part#" "53015-1010" (id 7) (at 271.78 144.78 0)
       (effects (font (size 1.27 1.27)) hide)
     )

Commit message: update bom2
Parts:
- U3: LCSC Part (none) -> C22429; MFR.Part# MC14049UBDTR2GOS -> CD4049UBDR; Manufacturer On Semi -> Texas Instruments; ODR.Part# MC14049UBDTR2GOS -> CD4049UBDR; Packaging 16-TSSOP (0.173", 4.40mm Width) -> SOIC-16; Supplier Digikey -> JLCPCB-Extended

Commit message: updates pdf.
Other:
- note added: "Parallel Side Input Hook"
- note added: "Parallel Side Output Hook"
- note removed: "Vend Side Pull Up Input"
- company: (none) -> Korean Paper Dispenser Parallel to Serial Module
- title: (none) -> Paper
Changed lines of the file:
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@@
 (kicad_sch (version 20210621) (generator eeschema)
   (paper "A4")
+  (title_block
+    (title "Paper")
+    (date "2021-07-30")
+    (rev "0.1")
+    (company "Korean Paper Dispenser Parallel to Serial Module")
+    (comment 1 "Features : 24V -> 12V, RS232, STM32G030")
+    (comment 2 "Proof of concept hardware for Rust-Embedded.")
+    (comment 3 "CERN-OHL-S-2.0")
+    (comment 4 "Jinwoo Park pmnxis@gmail.com")
+  )
   (junction (at 46.99 44.45) (diameter 0.9144) (color 0 0 0 0))
   (junction (at 46.99 91.44) (diameter 0.9144) (color 0 0 0 0))
@@
     (stroke (width 0) (type dash) (color 0 0 0 0))
   )
-  (text "Vend Side Pull Up Input" (at 19.05 20.32 0)
+  (text "Parallel Side Output Hook" (at 19.05 20.32 0)
     (effects (font (size 2.54 2.54)) (justify left bottom))
   )
@@
     (effects (font (size 1.27 1.27)) (justify right bottom))
   )
-  (text "Vend Side Pull Up Input" (at 77.47 20.32 0)
+  (text "Parallel Side Input Hook" (at 77.47 20.32 0)
     (effects (font (size 2.54 2.54)) (justify left bottom))
   )

Commit message: pre 2
Other:
- company: Korean Paper Dispenser Parallel to Serial Module -> Korean Paper Dispenser Parallel to Serial Adapter Module
Changed lines of the file:
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@@
     (date "2021-07-30")
     (rev "0.1")
-    (company "Korean Paper Dispenser Parallel to Serial Module")
+    (company "Korean Paper Dispenser Parallel to Serial Adapter Module")
     (comment 1 "Features : 24V -> 12V, RS232, STM32G030")
     (comment 2 "Proof of concept hardware for Rust-Embedded.")
@@
   (symbol (lib_id "power:+12V") (at 46.99 33.02 0) (unit 1)
     (in_bom yes) (on_board yes)
-    (property "Reference" "#PWR025" (id 0) (at 46.99 36.83 0)
+    (property "Reference" "#PWR026" (id 0) (at 46.99 36.83 0)
       (effects (font (size 1.27 1.27)) hide)
     )
@@
   (symbol (lib_id "power:+12V") (at 46.99 80.01 0) (unit 1)
     (in_bom yes) (on_board yes)
-    (property "Reference" "#PWR027" (id 0) (at 46.99 83.82 0)
+    (property "Reference" "#PWR028" (id 0) (at 46.99 83.82 0)
       (effects (font (size 1.27 1.27)) hide)
     )
@@
   (symbol (lib_id "power:+12V") (at 46.99 127 0) (unit 1)
     (in_bom yes) (on_board yes)
-    (property "Reference" "#PWR029" (id 0) (at 46.99 130.81 0)
+    (property "Reference" "#PWR030" (id 0) (at 46.99 130.81 0)
       (effects (font (size 1.27 1.27)) hide)
     )
@@
   (symbol (lib_id "power:+12V") (at 92.71 34.29 0) (unit 1)
     (in_bom yes) (on_board yes)
-    (property "Reference" "#PWR034" (id 0) (at 92.71 38.1 0)
+    (property "Reference" "#PWR035" (id 0) (at 92.71 38.1 0)
       (effects (font (size 1.27 1.27)) hide)
     )
@@
   (symbol (lib_id "power:+12V") (at 92.71 76.2 0) (unit 1)
     (in_bom yes) (on_board yes)
-    (property "Reference" "#PWR035" (id 0) (at 92.71 80.01 0)
+    (property "Reference" "#PWR036" (id 0) (at 92.71 80.01 0)
       (effects (font (size 1.27 1.27)) hide)
     )
@@
   (symbol (lib_id "power:+12V") (at 92.71 118.11 0) (unit 1)
     (in_bom yes) (on_board yes)
-    (property "Reference" "#PWR036" (id 0) (at 92.71 121.92 0)
+    (property "Reference" "#PWR037" (id 0) (at 92.71 121.92 0)
       (effects (font (size 1.27 1.27)) hide)
     )
@@
   (symbol (lib_id "power:+3V3") (at 111.76 158.75 0) (unit 1)
     (in_bom yes) (on_board yes)
-    (property "Reference" "#PWR040" (id 0) (at 111.76 162.56 0)
+    (property "Reference" "#PWR041" (id 0) (at 111.76 162.56 0)
       (effects (font (size 1.27 1.27)) hide)
     )
@@
   (symbol (lib_id "power:+12V") (at 265.43 148.59 90) (unit 1)
     (in_bom yes) (on_board yes)
-    (property "Reference" "#PWR044" (id 0) (at 269.24 148.59 0)
+    (property "Reference" "#PWR045" (id 0) (at 269.24 148.59 0)
       (effects (font (size 1.27 1.27)) hide)
     )
@@
   (symbol (lib_id "power:GND") (at 46.99 63.5 0) (unit 1)
     (in_bom yes) (on_board yes)
-    (property "Reference" "#PWR026" (id 0) (at 46.99 69.85 0)
+    (property "Reference" "#PWR027" (id 0) (at 46.99 69.85 0)
       (effects (font (size 1.27 1.27)) hide)
     )
@@
   (symbol (lib_id "power:GND") (at 46.99 110.49 0) (unit 1)
     (in_bom yes) (on_board yes)
-    (property "Reference" "#PWR028" (id 0) (at 46.99 116.84 0)
+    (property "Reference" "#PWR029" (id 0) (at 46.99 116.84 0)
       (effects (font (size 1.27 1.27)) hide)
     )
@@
   (symbol (lib_id "power:GND") (at 46.99 157.48 0) (unit 1)
     (in_bom yes) (on_board yes)
-    (property "Reference" "#PWR030" (id 0) (at 46.99 163.83 0)
+    (property "Reference" "#PWR031" (id 0) (at 46.99 163.83 0)
       (effects (font (size 1.27 1.27)) hide)
     )
@@
   (symbol (lib_id "power:GND") (at 83.82 160.02 270) (unit 1)
     (in_bom yes) (on_board yes) (fields_autoplaced)
-    (property "Reference" "#PWR031" (id 0) (at 77.47 160.02 0)
+    (property "Reference" "#PWR032" (id 0) (at 77.47 160.02 0)
       (effects (font (size 1.27 1.27)) hide)
     )
@@
   (symbol (lib_id "power:GND") (at 83.82 172.72 270) (unit 1)
     (in_bom yes) (on_board yes) (fields_autoplaced)
-    (property "Reference" "#PWR032" (id 0) (at 77.47 172.72 0)
+    (property "Reference" "#PWR033" (id 0) (at 77.47 172.72 0)
       (effects (font (size 1.27 1.27)) hide)
     )
@@
   (symbol (lib_id "power:GND") (at 83.82 185.42 270) (unit 1)
     (in_bom yes) (on_board yes) (fields_autoplaced)
-    (property "Reference" "#PWR033" (id 0) (at 77.47 185.42 0)
+    (property "Reference" "#PWR034" (id 0) (at 77.47 185.42 0)
       (effects (font (size 1.27 1.27)) hide)
     )
@@
   (symbol (lib_id "power:GND") (at 102.87 57.15 0) (unit 1)
     (in_bom yes) (on_board yes)
-    (property "Reference" "#PWR037" (id 0) (at 102.87 63.5 0)
+    (property "Reference" "#PWR038" (id 0) (at 102.87 63.5 0)
       (effects (font (size 1.27 1.27)) hide)
     )
@@
   (symbol (lib_id "power:GND") (at 102.87 99.06 0) (unit 1)
     (in_bom yes) (on_board yes)
-    (property "Reference" "#PWR038" (id 0) (at 102.87 105.41 0)
+    (property "Reference" "#PWR039" (id 0) (at 102.87 105.41 0)
       (effects (font (size 1.27 1.27)) hide)
     )
@@
   (symbol (lib_id "power:GND") (at 102.87 140.97 0) (unit 1)
     (in_bom yes) (on_board yes)
-    (property "Reference" "#PWR039" (id 0) (at 102.87 147.32 0)
+    (property "Reference" "#PWR040" (id 0) (at 102.87 147.32 0)
       (effects (font (size 1.27 1.27)) hide)
     )
@@
   (symbol (lib_id "power:GND") (at 111.76 184.15 0) (unit 1)
     (in_bom yes) (on_board yes)
-    (property "Reference" "#PWR041" (id 0) (at 111.76 190.5 0)
+    (property "Reference" "#PWR042" (id 0) (at 111.76 190.5 0)
       (effects (font (size 1.27 1.27)) hide)
     )
@@
   (symbol (lib_id "power:GND") (at 264.16 152.4 270) (unit 1)
     (in_bom yes) (on_board yes)
-    (property "Reference" "#PWR042" (id 0) (at 257.81 152.4 0)
+    (property "Reference" "#PWR043" (id 0) (at 257.81 152.4 0)
       (effects (font (size 1.27 1.27)) hide)
     )
@@
   (symbol (lib_id "power:GND") (at 264.16 154.94 270) (unit 1)
     (in_bom yes) (on_board yes)
-    (property "Reference" "#PWR043" (id 0) (at 257.81 154.94 0)
-      (effects (font (size 1.27 1.27)) hide)
-    )
+    (property "Reference" "#PWR044" (id 0) (at 257.81 154.94 0)
+      (effects (font (size 1.27 1.27)) hide)
+    )

Commit message: release/v3 update
Parts:
- R3, R4, R5: value 4.7k -> 8.2k; LCSC Part C25900 -> C25924; MFR.Part# 0402WGF4701TCE -> 0402WGF8201TCE; ODR.Part# RES 4.7k 1005 -> RES 8.2k 1005
- R6, R7, R8: value 4.7k -> 27k; LCSC Part C25900 -> C25771; MFR.Part# 0402WGF4701TCE -> 0402WGF2702TCE; ODR.Part# RES 4.7k 1005 -> RES 27k 1005; now left out of the parts list
Connections:
- net +12V: now also J2.7 (Pin_7), J2.8 (Pin_8); no longer J2.3 (Pin_3), J2.4 (Pin_4)
- net GND: now also J2.10 (Pin_10), J2.9 (Pin_9), U3.11, U3.14, U3.9; no longer J2.1 (Pin_1), J2.2 (Pin_2), U3.3, U3.5, U3.7
- net J_EMPTY: now also J2.5 (Pin_5); no longer J2.6 (Pin_6)
- net J_ERROR: now also J2.6 (Pin_6); no longer J2.5 (Pin_5)
- net J_INHIBIT: now also J2.1 (Pin_1); no longer J2.10 (Pin_10)
- net J_OUT_PULSE: now also J2.4 (Pin_4); no longer J2.7 (Pin_7)
- net J_PULSE: now also J2.3 (Pin_3); no longer J2.8 (Pin_8)
- net J_RESET: now also J2.2 (Pin_2); no longer J2.9 (Pin_9)
- net P_EMPTY: now also U3.4; no longer U3.12
- net P_ERROR: now also U3.6; no longer U3.10
- net P_OUT_PULSE: now also U3.2; no longer U3.15
- net at C9.1, R9.2: now also U3.3; no longer U3.14
- net at C11.1, R11.2: now also U3.7; no longer U3.9
- net at C10.1, R10.2: now also U3.5; no longer U3.11
Other:
- note added: "OBDL-1000P serve 5v-4.7k Pull-up already. By V=IR, I servce a 27k"
- moved on the sheet: U3A, U3B, U3C, U3D, U3E, U3F
