File: Power.kicad_sch (KiCad schematic)
At the start: 28 parts, among them U2 RT8259GJ6, U3 TPS5430DDA

Commit message: v1
Parts:
- added C19: 10uF 50V, Capacitor_SMD:C_1206_3216Metric, symbol Device:C
- renumbered C16 to C13, C17 to C14, C18 to C15, C19 to C16, C20 to C17, C21 to C18, C22 to C20, C23 to C21, C24 to C22, C25 to C23, C26 to C24, C27 to C25, C28 to C26, C29 to C27, C30 to C28, D1 to D3, D2 to D4, D3 to D5, R22 to R12, R23 to R13, R24 to R14, R25 to R15, R26 to R16, R27 to R17, U2 to U4, U3 to U5
Connections:
- net +24V: now also C19.1
- net GND: now also C19.2

Commit message: update bom
Parts:
- D3: value LED_RED -> LED GREEN; LCSC Part C84256 -> C2297; MFR.Part# FC-2012HRK-620D -> KT-0805G; ODR.Part# LED RED 2012 -> LED GREEN 2012
- D4: LCSC Part (none) -> C134441; MFR.Part# (none) -> B240AQ-13-F; Manufacturer (none) -> Diodes Incorporated; Mount (none) -> SMD; ODR.Part# (none) -> B240AQ-13-F; Packaging (none) -> SMA(DO-214AC); Supplier (none) -> JLCPCB-Extended
- D5: LCSC Part (none) -> C155302; MFR.Part# (none) -> MBRD20200CT-13; Manufacturer (none) -> Diodes Incorporated; Mount (none) -> SMD; ODR.Part# (none) -> MBRD20200CT-13; Packaging (none) -> TO-252-2; Supplier (none) -> JLCPCB-Extended
- L2: value MCF-1040-330-N2 -> MWSA1206S-330MT; footprint Inductor_SMD:L_12x12mm_H6mm -> Power_Inductor_Extended:L_Sunlord-MWSA1206S; LCSC Part C307880 -> C408530; MFR.Part# VLS6045EX-4R7M -> MWSA1206S-330MT; ODR.Part# 33uH 4A -> 33uH 5.5A; Packaging L_6.0*6.0*4.5 -> L_12.6*13.45*5.8
Changed lines of the file:
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@@
     (in_bom yes) (on_board yes)
     (property "Reference" "L2" (id 0) (at 121.92 35.56 90))
-    (property "Value" "MCF-1040-330-N2" (id 1) (at 127 38.1 90)
+    (property "Value" "MWSA1206S-330MT" (id 1) (at 127 38.1 90)
       (effects (font (size 1 1)))
     )
-    (property "Footprint" "Inductor_SMD:L_12x12mm_H6mm" (id 2) (at 137.16 41.91 90)
-      (effects (font (size 1.27 1.27)) hide)
-    )
-    (property "Datasheet" "https://product.tdk.com/en/system/files?file=dam/doc/product/inductor/inductor/smd/catalog/inductor_commercial_power_vls6045ex_en.pdf" (id 3) (at 124.46 40.64 0)
-      (effects (font (size 1.27 1.27)) hide)
-    )
-    (property "MFR.Part#" "VLS6045EX-4R7M" (id 4) (at 125.73 41.91 90)
-      (effects (font (size 1.27 1.27)) hide)
-    )
-    (property "ODR.Part#" "33uH 4A" (id 5) (at 130.81 35.56 90)
+    (property "Footprint" "Power_Inductor_Extended:L_Sunlord-MWSA1206S" (id 2) (at 137.16 41.91 90)
+      (effects (font (size 1.27 1.27)) hide)
+    )
+    (property "Datasheet" "https://datasheet.lcsc.com/lcsc/1912111437_Sunlord-MWSA1206S-330MT_C408530.pdf" (id 3) (at 124.46 40.64 0)
+      (effects (font (size 1.27 1.27)) hide)
+    )
+    (property "MFR.Part#" "MWSA1206S-330MT" (id 4) (at 125.73 41.91 90)
+      (effects (font (size 1.27 1.27)) hide)
+    )
+    (property "ODR.Part#" "33uH 5.5A" (id 5) (at 130.81 35.56 90)
       (effects (font (size 0.8382 0.8382)))
     )
-    (property "Packaging" "L_6.0*6.0*4.5" (id 6) (at 125.73 41.91 90)
+    (property "Packaging" "L_12.6*13.45*5.8" (id 6) (at 125.73 41.91 90)
       (effects (font (size 1.27 1.27)) hide)
     )
@@
       (effects (font (size 1.27 1.27)) hide)
     )
-    (property "LCSC Part" "C307880" (id 8) (at 127 41.91 90)
+    (property "LCSC Part" "C408530" (id 8) (at 127 41.91 90)
       (effects (font (size 1.27 1.27)) hide)
     )
@@
       (effects (font (size 1.27 1.27)) hide)
     )
-    (property "Datasheet" "http://www.jameco.com/Jameco/Products/ProdDS/1538777.pdf" (id 3) (at 99.06 120.65 0)
+    (property "Datasheet" "https://www.diodes.com/assets/Datasheets/B220AQ-Q-B260AQ-Q.pdf" (id 3) (at 99.06 120.65 0)
+      (effects (font (size 1.27 1.27)) hide)
+    )
+    (property "LCSC Part" "C134441" (id 4) (at 99.06 120.65 0)
+      (effects (font (size 1.27 1.27)) hide)
+    )
+    (property "MFR.Part#" "B240AQ-13-F" (id 5) (at 99.06 120.65 0)
+      (effects (font (size 1.27 1.27)) hide)
+    )
+    (property "Manufacturer" "Diodes Incorporated" (id 6) (at 99.06 120.65 0)
+      (effects (font (size 1.27 1.27)) hide)
+    )
+    (property "Mount" "SMD" (id 7) (at 99.06 120.65 0)
+      (effects (font (size 1.27 1.27)) hide)
+    )
+    (property "ODR.Part#" "B240AQ-13-F" (id 8) (at 99.06 120.65 0)
+      (effects (font (size 1.27 1.27)) hide)
+    )
+    (property "Packaging" "SMA(DO-214AC)" (id 9) (at 99.06 120.65 0)
+      (effects (font (size 1.27 1.27)) hide)
+    )
+    (property "Supplier" "JLCPCB-Extended" (id 10) (at 99.06 120.65 0)
       (effects (font (size 1.27 1.27)) hide)
     )
@@
       (effects (font (size 1.27 1.27)) hide)
     )
-    (property "Datasheet" "http://www.jameco.com/Jameco/Products/ProdDS/1538777.pdf" (id 3) (at 116.84 52.07 0)
+    (property "Datasheet" "https://www.diodes.com/assets/Datasheets/MBRD20200CT.pdf" (id 3) (at 116.84 52.07 0)
+      (effects (font (size 1.27 1.27)) hide)
+    )
+    (property "LCSC Part" "C155302" (id 4) (at 116.84 52.07 0)
+      (effects (font (size 1.27 1.27)) hide)
+    )
+    (property "MFR.Part#" "MBRD20200CT-13" (id 5) (at 116.84 52.07 0)
+      (effects (font (size 1.27 1.27)) hide)
+    )
+    (property "Manufacturer" "Diodes Incorporated" (id 6) (at 116.84 52.07 0)
+      (effects (font (size 1.27 1.27)) hide)
+    )
+    (property "Mount" "SMD" (id 7) (at 116.84 52.07 0)
+      (effects (font (size 1.27 1.27)) hide)
+    )
+    (property "ODR.Part#" "MBRD20200CT-13" (id 8) (at 116.84 52.07 0)
+      (effects (font (size 1.27 1.27)) hide)
+    )
+    (property "Packaging" "TO-252-2" (id 9) (at 116.84 52.07 0)
+      (effects (font (size 1.27 1.27)) hide)
+    )
+    (property "Supplier" "JLCPCB-Extended" (id 10) (at 116.84 52.07 0)
       (effects (font (size 1.27 1.27)) hide)
     )
@@
     (in_bom yes) (on_board yes)
     (property "Reference" "D3" (id 0) (at 62.4078 135.763 0))
-    (property "Value" "LED_RED" (id 1) (at 62.4078 138.0744 0))
+    (property "Value" "LED GREEN" (id 1) (at 62.4078 138.0744 0))
     (property "Footprint" "LED_SMD:LED_0805_2012Metric" (id 2) (at 62.23 142.24 0)
       (effects (font (size 1.27 1.27)) hide)
     )
-    (property "Datasheet" "Foshan-NationStar-Optoelectronics-FC-2012HRK-620D_C84256.pdf" (id 3) (at 62.23 142.24 0)
-      (effects (font (size 1.27 1.27)) hide)
-    )
-    (property "LCSC Part" "C84256" (id 4) (at 62.23 142.24 0)
-      (effects (font (size 1.27 1.27)) hide)
-    )
-    (property "MFR.Part#" "FC-2012HRK-620D" (id 5) (at 62.23 142.24 0)
+    (property "Datasheet" "https://datasheet.lcsc.com/lcsc/1806151820_Hubei-KENTO-Elec-C2297_C2297.pdf" (id 3) (at 62.23 142.24 0)
+      (effects (font (size 1.27 1.27)) hide)
+    )
+    (property "LCSC Part" "C2297" (id 4) (at 62.23 142.24 0)
+      (effects (font (size 1.27 1.27)) hide)
+    )
+    (property "MFR.Part#" "KT-0805G" (id 5) (at 62.23 142.24 0)
       (effects (font (size 1.27 1.27)) hide)
     )
@@
       (effects (font (size 1.27 1.27)) hide)
     )
-    (property "ODR.Part#" "LED RED 2012" (id 8) (at 62.23 142.24 0)
-      (effects (font (size 1.27 1.27)) hide)
-    )
+    (property "ODR.Part#" "LED GREEN 2012" (id 8) (at 62.23 142.24 0)
+      (effects (font (size 1.27 1.27)) hide)
+    )

Commit message: update bom2
Parts:
- R17: ODR.Part# RES 10k 1% 1608 -> RES 1.13k 1% 1608
- U5: MFR.Part# (none) -> C9864; Manufacturer (none) -> Texas Instruments; Mount (none) -> SMD; ODR.Part# (none) -> TPS5430DDAR; Packaging (none) -> LSOP-8_EP_3.9x4.9x1.27P; Supplier (none) -> JLCPCB-Basic
Changed lines of the file:
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@@
       (effects (font (size 1.27 1.27)) hide)
     )
-    (property "ODR.Part#" "RES 10k 1% 1608" (id 4) (at 203.2 57.7849 0)
+    (property "ODR.Part#" "RES 1.13k 1% 1608" (id 4) (at 203.2 57.7849 0)
       (effects (font (size 0.8382 0.8382)) (justify left))
     )
@@
       (effects (font (size 1.27 1.27)) hide)
     )
+    (property "MFR.Part#" "C9864" (id 4) (at 92.71 45.72 0)
+      (effects (font (size 1.27 1.27)) hide)
+    )
+    (property "Manufacturer" "Texas Instruments" (id 5) (at 92.71 45.72 0)
+      (effects (font (size 1.27 1.27)) hide)
+    )
+    (property "Mount" "SMD" (id 6) (at 92.71 45.72 0)
+      (effects (font (size 1.27 1.27)) hide)
+    )
+    (property "ODR.Part#" "TPS5430DDAR" (id 7) (at 92.71 45.72 0)
+      (effects (font (size 1.27 1.27)) hide)
+    )
+    (property "Packaging" "LSOP-8_EP_3.9x4.9x1.27P" (id 8) (at 92.71 45.72 0)
+      (effects (font (size 1.27 1.27)) hide)
+    )
+    (property "Supplier" "JLCPCB-Basic" (id 9) (at 92.71 45.72 0)
+      (effects (font (size 1.27 1.27)) hide)
+    )

Commit message: updates pdf.
Other:
- company: (none) -> Korean Paper Dispenser Parallel to Serial Module
- title: (none) -> Power Domain
Changed lines of the file:
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@@
 (kicad_sch (version 20210621) (generator eeschema)
   (paper "A4")
+  (title_block
+    (title "Power Domain")
+    (date "2021-07-30")
+    (rev "0.1")
+    (company "Korean Paper Dispenser Parallel to Serial Module")
+    (comment 1 "Features : 24V -> 12V, RS232, STM32G030")
+    (comment 2 "Proof of concept hardware for Rust-Embedded.")
+    (comment 3 "CERN-OHL-S-2.0")
+    (comment 4 "Jinwoo Park pmnxis@gmail.com")
+  )
   (junction (at 35.56 107.95) (diameter 0.9144) (color 0 0 0 0))
   (junction (at 38.1 40.64) (diameter 0.9144) (color 0 0 0 0))

Commit message: pre 2
Parts:
- added C18, C20: 100nF, Capacitor_SMD:C_0402_1005Metric, symbol Device:C
- added C27, C28: 10uF 50V, Capacitor_SMD:C_1206_3216Metric, symbol Device:C
- D4: renamed from D5; symbol Diode:B330 -> Device:D_Schottky_AKA
- D5: renamed from D4; symbol Diode:B330 -> Diode:B240
- renumbered C14 to C13, C15 to C14, C17 to C15, C18 to C16, C19 to C17, C21 to C19, C13 to C21, C23 to C22, C25 to C23, C26 to C24, C27 to C25, C28 to C26, C16 to C29, C20 to C30, C22 to C31, C24 to C32, D3 to D6, L2 to L1, L1 to L2, R16 to R12, R17 to R13, R13 to R14, R14 to R15, R15 to R16, R12 to R17, U5 to U4, U4 to U5
Connections:
- net +12V: now also C20.1, C27.1, C28.1
- net +24V: now also C18.1
- net BIG_PH: now also D4.2 (K); no longer D4.1 (K)
- net GND: now also D4.1 (A), D4.3 (A), C18.2, C20.2, C27.2, C28.2; no longer D4.2 (A)
Other:
- note added: "- Alternative - MBRD20150CT-13 (LCSC:C151357)"
- note added: "24V to 12V : Switching Regulator"
- company: Korean Paper Dispenser Parallel to Serial Module -> Korean Paper Dispenser Parallel to Serial Adapter Module
- moved on the sheet: C13, C14, C15, C16, C17, C19, C21, C23, C24, C25, C26, C29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

Commit message: release/v3 update
Parts:
- removed C13, C14, C16, C22, C23, C24, C25, C26, C27: 10uF 50V, Capacitor_SMD:C_1206_3216Metric, symbol Device:C
- removed U4: TPS5430DDA, Package_SO:TI_SO-PowerPAD-8_ThermalVias, symbol Regulator_Switching:TPS5430DDA
- added C13, C14: 68uF, Capacitor_SMD:CP_Elec_8x10, symbol Device:C_Polarized_Small
- added C19, C20: 100uF, Capacitor_SMD:CP_Elec_8x6.9, symbol Device:C_Polarized_Small
- added R14: 20k, Resistor_SMD:R_0603_1608Metric, symbol Device:R_US
- added U4: LMR14050SDDA, Package_SO:TI_SO-PowerPAD-8_ThermalVias, symbol Regulator_Switching_Extended:LMR14050SDDA
- C15: value 10uF 50V -> 330pF; footprint Capacitor_SMD:C_1206_3216Metric -> Capacitor_SMD:C_0603_1608Metric; LCSC Part C13585 -> C1664; MFR.Part# CL31A106KBHNNNE -> CL10C331JB8NNNC; Manufacturer SAMSUNG -> ANY; ODR.Part# CAP 10uF 50V 3216 -> CAP 330pF 1608; Packaging 3216 -> 1608
- C16: renamed from C18; value 100nF -> 100nF 50V; footprint Capacitor_SMD:C_0402_1005Metric -> Capacitor_SMD:C_0603_1608Metric; LCSC Part C1525 -> C14663; MFR.Part# CL05B104KO5NNNC -> CC0603KRX7R9BB104; ODR.Part# CAP 100nF 1005 -> CAP 100nF 50V 1608; Packaging 1005 -> 1608
- C17: value 10uF 50V -> 22nF; footprint Capacitor_SMD:C_1206_3216Metric -> Capacitor_SMD:C_0603_1608Metric; LCSC Part C13585 -> C21122; MFR.Part# CL31A106KBHNNNE -> CL10B223KB8NNNC; Manufacturer SAMSUNG -> ANY; ODR.Part# CAP 10uF 50V 3216 -> CAP 22nF 1608; Packaging 3216 -> 1608
- C18: renamed from C19; value 10nF -> 100nF 50V; footprint Capacitor_SMD:C_0402_1005Metric -> Capacitor_SMD:C_0603_1608Metric; LCSC Part C15195 -> C14663; MFR.Part# CL05B103KB5NNNC -> CC0603KRX7R9BB104; ODR.Part# CAP 10nF 1005 -> CAP 100nF 50V 1608; Packaging 1005 -> 1608
- C21: value 10uF 50V -> 100nF 50V; footprint Capacitor_SMD:C_1206_3216Metric -> Capacitor_SMD:C_0603_1608Metric; LCSC Part C13585 -> C14663; MFR.Part# CL31A106KBHNNNE -> CC0603KRX7R9BB104; Manufacturer SAMSUNG -> ANY; ODR.Part# CAP 10uF 50V 3216 -> CAP 100nF 50V 1608; Packaging 3216 -> 1608
- C23: renamed from C20; value 100nF -> 100nF 50V; footprint Capacitor_SMD:C_0402_1005Metric -> Capacitor_SMD:C_0603_1608Metric; LCSC Part C1525 -> C14663; MFR.Part# CL05B104KO5NNNC -> CC0603KRX7R9BB104; ODR.Part# CAP 100nF 1005 -> CAP 100nF 50V 1608; Packaging 1005 -> 1608
- C24: renamed from C29; value 100nF -> 100nF 50V; footprint Capacitor_SMD:C_0402_1005Metric -> Capacitor_SMD:C_0603_1608Metric; LCSC Part C1525 -> C14663; MFR.Part# CL05B104KO5NNNC -> CC0603KRX7R9BB104; ODR.Part# CAP 100nF 1005 -> CAP 100nF 50V 1608; Packaging 1005 -> 1608
- D4: value MBRD20200CT-13 -> MBRD20150CT-13; LCSC Part C155302 -> C151357; MFR.Part# MBRD20200CT-13 -> MBRD20150CT-13; ODR.Part# MBRD20200CT-13 -> MBRD20150CT-13
- L1: value MWSA1206S-330MT -> SPM10040T-4R7M; footprint Power_Inductor_Extended:L_Sunlord-MWSA1206S -> TDK-SPM10040:L_TDK_SPM10040; LCSC Part C408530 -> C138681; MFR.Part# MWSA1206S-330MT -> SPM10040T-4R7M; Manufacturer Taiyo Yuden -> TDK; ODR.Part# 33uH 5.5A -> 4.7A 8A; Packaging L_12.6*13.45*5.8 -> L_12.5*12.5*7.5
- R12: renamed from R13; value 1.13k -> 150k; LCSC Part C22833 -> C22807; MFR.Part# 0603WAF1131T5E -> 0603WAF1503T5E; ODR.Part# RES 1.13k 1% 1608 -> RES 150k 1% 1608
- R13: renamed from R12; value 10k -> 10k 0.1W; LCSC Part C22833 -> C25804; MFR.Part# 0603WAF1131T5E -> 0603WAF1002T5E
- R18: renamed from R17; value 4.7k -> 10k 0.1W; footprint Resistor_SMD:R_0402_1005Metric -> Resistor_SMD:R_0603_1608Metric; LCSC Part C25900 -> C25804; MFR.Part# 0402WGF4701TCE -> 0603WAF1002T5E; ODR.Part# RES 4.7k 1005 -> RES 10k 1% 1608; Packaging 1005 -> 1608
- renumbered C28 to C22, C30 to C25, C31 to C26, C32 to C27, R14 to R15, R15 to R16, R16 to R17
Connections:
- net +12V: now also C15.1, R12.1, C19.1, C20.1; no longer R13.1
- net +24V: now also C13.1, C14.1, U4.2 (VIN), U4.3 (EN); no longer C15.1, C17.1
- net GND: now also R13.2, C13.2, C14.2, C19.2, C20.2, R14.2, U4.7 (GND), U4.9 (EP); no longer C15.2, R12.2
- net BIG_BOOT: now reaches C18.1
- net BIG_BOOT: now also U4.1 (BOOT)
- net BIG_PH renamed BIG_SW
- net BIG_SW: now also U4.8 (SW)
- removed net BIG_VS: R12.1, R13.2
- new net BIG_FB: C15.2, R12.2, R13.1, U4.5 (FB)
- new net BIG_RTS: R14.1, U4.4 (RT/SYNC)
- new net BIG_SS: C17.1, U4.6 (SS)
- no-connect marks 1 -> 0
Other:
- note added: "- More Stronger - MBRD20200CT-13"
- note added: "Soft Start 5msecs"
- note removed: "- Alternative - MBRD20150CT-13 (LCSC:C151357)"
- moved on the sheet: C16, C22, C23, D4, R12, R13, R15, R16, R17
